File: hardware/comms/02_link.kicad_sch (KiCad schematic)
At the start: 21 parts, among them Q1 MMBT3904, U4 ST60A3H1, U5 PTN3222GM, U6 TXS0108E

Commit message: Rev A after review: ST's antenna ground, 1.8 V rail, pull-ups, 90 ohm pairs
Two independent reviews (schematic against the data sheets, layout
against JLCPCB's limits and ST's B2379A) found no blocker and a dozen
things worth fixing. The board is regenerated and routed again.

Layout: the ST60's ball field is laid as ST lays it -- nine signals
straight out through one side of the ring, the supply along the top --
and the island and fence vias are ST's own, from its drill file (33 and
45 fit, where rev A had 13 and 15). USB pairs on the back 0.28/0.16 mm;
the +1V8 plane redrawn so the pair to the repeater has +3V3 under it
throughout. ST60 mask openings 0.30 mm. Silkscreen to JLCPCB's sizes.
VBUS joined on the back, not under the USB-C shell. Three fiducials.

Schematic: 1.8 uF on +1V8 and its enable pulled down; 4k7 on MODE_INT;
4k7 pull-ups on the 1.8 V side of the four I2C lines; 220 R on the LEDs.

README has the review table, what was left as it is, and ordering notes
(Standard PCBA, 0.10 mm stencil, nylon standoffs, firmware sequencing).

Co-Authored-By: Claude Fable 5.1 <noreply@anthropic.com>
Parts:
- removed C23: 1u, Capacitor_SMD:C_0402_1005Metric, symbol Device:C
- added R24, R25, R26, R27, R31: 4k7, Resistor_SMD:R_0402_1005Metric, symbol Device:R
- C26: value 1u -> 470n
- R30: value 1k -> 220R
Connections:
- net +1V8: now also R24.2, R25.2, R26.2, R27.2
- net GND: now also R31.2
- net ST_G2: now also R26.1
- net ST_G3: now also R27.1
- net ST_MODE_INT: now also R31.1
- net ST_SCL: now also R24.1
- net ST_SDA: now also R25.1
Other:
- note added: "After ST's X-NUCLEO-60K1A1 (B2379A): the ST60A3H1 on +1V8 through a 0 R link, the PTN3222 on its eUSB2 pair and held in reset by LINK_STATUS, an eight-channel auto-direction translator to 3.3 V (TXS0108E here, ST2378E there), RF_EN by divider, the link LED off an NPN. The translator is off (LS_OE low) until the RP2350 enables it, so the ST60 powers up with its own straps on its pins and R31 on MO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"
- note removed: "After ST's X-NUCLEO-60K1A1 (B2379A): the ST60A3H1 on +1V8 through a 0 R link, the PTN3222 on its eUSB2 pair and held in reset by LINK_STATUS, an eight-channel auto-direction translator to 3.3 V (TXS0108E here, ST2378E there), RF_EN by divider, the link LED off an NPN. The translator is off (LS_OE low) until the RP2350 enables it, so the ST60 powers up with only its own straps on its pins. No pull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"
