File: hardware/comms/03_usb_power.kicad_sch (KiCad schematic)
At the start: 20 parts, among them J1 USB-C, U10 TS3USB221A, U2 AMS1117-3.3, U7 TLV75518P, U8 USBLC6-2SC6, U9 TS3USB221A

Commit message: Rev A after review: ST's antenna ground, 1.8 V rail, pull-ups, 90 ohm pairs
Two independent reviews (schematic against the data sheets, layout
against JLCPCB's limits and ST's B2379A) found no blocker and a dozen
things worth fixing. The board is regenerated and routed again.

Layout: the ST60's ball field is laid as ST lays it -- nine signals
straight out through one side of the ring, the supply along the top --
and the island and fence vias are ST's own, from its drill file (33 and
45 fit, where rev A had 13 and 15). USB pairs on the back 0.28/0.16 mm;
the +1V8 plane redrawn so the pair to the repeater has +3V3 under it
throughout. ST60 mask openings 0.30 mm. Silkscreen to JLCPCB's sizes.
VBUS joined on the back, not under the USB-C shell. Three fiducials.

Schematic: 1.8 uF on +1V8 and its enable pulled down; 4k7 on MODE_INT;
4k7 pull-ups on the 1.8 V side of the four I2C lines; 220 R on the LEDs.

README has the review table, what was left as it is, and ordering notes
(Standard PCBA, 0.10 mm stencil, nylon standoffs, firmware sequencing).

Co-Authored-By: Claude Fable 5.1 <noreply@anthropic.com>
Parts:
- R14: value 1k -> 220R
- R15: value 10k -> 4k7
Connections:
- net +3V3: no longer R15.1
- net GND: now also R15.1
Other:
- moved on the sheet: R15
Changed lines of the file:
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@@
 			(at 149.6060 151.1300 0)
 			(effects (font (size 1.27 1.27)) (justify left)))
-		(property "Value" "1k"
+		(property "Value" "220R"
 			(at 149.6060 153.6700 0)
 			(effects (font (size 1.27 1.27)) (justify left)))
@@
 	(symbol
 		(lib_id "Device:R")
-		(at 241.3000 149.8600 0)
+		(at 243.8400 166.3700 180)
 		(unit 1)
 		(exclude_from_sim no)
@@
 		(dnp no)
 		(property "Reference" "R15"
-			(at 243.5860 148.5900 0)
-			(effects (font (size 1.27 1.27)) (justify left)))
-		(property "Value" "10k"
-			(at 243.5860 151.1300 0)
-			(effects (font (size 1.27 1.27)) (justify left)))
-		(property "Footprint" "Resistor_SMD:R_0402_1005Metric" (at 241.3000 149.8600 0)
-			(effects (font (size 1.27 1.27)) (hide yes)))
-		(property "Datasheet" "~" (at 241.3000 149.8600 0)
+			(at 246.1260 165.1000 0)
+			(effects (font (size 1.27 1.27)) (justify right)))
+		(property "Value" "4k7"
+			(at 246.1260 167.6400 0)
+			(effects (font (size 1.27 1.27)) (justify right)))
+		(property "Footprint" "Resistor_SMD:R_0402_1005Metric" (at 243.8400 166.3700 0)
+			(effects (font (size 1.27 1.27)) (hide yes)))
+		(property "Datasheet" "~" (at 243.8400 166.3700 0)
 			(effects (font (size 1.27 1.27)) (hide yes)))
 		(pin "1")
@@
 	(symbol
 		(lib_id "power:GND")
+		(at 243.8400 170.1800 0)
+		(unit 1)
+		(exclude_from_sim no)
+		(in_bom yes)
+		(on_board yes)
+		(dnp no)
+		(property "Reference" "#PWR4028" (at 243.8400 170.1800 0)
+			(effects (font (size 1.27 1.27)) (hide yes)))
+		(property "Value" "GND" (at 243.8400 173.9900 0)
+			(effects (font (size 1.27 1.27))))
+		(property "Footprint" "" (at 243.8400 170.1800 0)
+			(effects (font (size 1.27 1.27)) (hide yes)))
+		(pin "1")
+		(instances (project "comms" (path "/8132f9b4-61be-5b7f-9744-e0828e24db53/d481352e-8ed5-5537-86a1-5b377647b88b" (reference "#PWR4028") (unit 1))))
+	)
+	(symbol
+		(lib_id "power:GND")
 		(at 284.4800 153.6700 0)
 		(unit 1)
@@
 		(on_board yes)
 		(dnp no)
-		(property "Reference" "#PWR4028" (at 284.4800 153.6700 0)
+		(property "Reference" "#PWR4029" (at 284.4800 153.6700 0)
 			(effects (font (size 1.27 1.27)) (hide yes)))
 		(property "Value" "GND" (at 284.4800 157.4800 0)
@@
 			(effects (font (size 1.27 1.27)) (hide yes)))
 		(pin "1")
-		(instances (project "comms" (path "/8132f9b4-61be-5b7f-9744-e0828e24db53/d481352e-8ed5-5537-86a1-5b377647b88b" (reference "#PWR4028") (unit 1))))
+		(instances (project "comms" (path "/8132f9b4-61be-5b7f-9744-e0828e24db53/d481352e-8ed5-5537-86a1-5b377647b88b" (reference "#PWR4029") (unit 1))))
 	)
 	(symbol
@@
 	(wire (pts (xy 218.4400 146.0500) (xy 228.6000 146.0500))
 		(stroke (width 0) (type default)))
-	(wire (pts (xy 228.6000 146.0500) (xy 241.3000 146.0500))
-		(stroke (width 0) (type default)))
-	(wire (pts (xy 241.3000 146.0500) (xy 256.5400 146.0500))
-		(stroke (width 0) (type default)))
-	(wire (pts (xy 241.3000 153.6700) (xy 251.4600 153.6700))
-		(stroke (width 0) (type default)))
-	(wire (pts (xy 251.4600 148.5900) (xy 251.4600 153.6700))
+	(wire (pts (xy 228.6000 146.0500) (xy 256.5400 146.0500))
+		(stroke (width 0) (type default)))
+	(wire (pts (xy 243.8400 162.5600) (xy 251.4600 162.5600))
+		(stroke (width 0) (type default)))
+	(wire (pts (xy 251.4600 148.5900) (xy 251.4600 162.5600))
 		(stroke (width 0) (type default)))
 	(wire (pts (xy 251.4600 148.5900) (xy 256.5400 148.5900))
 		(stroke (width 0) (type default)))
-	(wire (pts (xy 241.3000 153.6700) (xy 241.3000 156.2100))
+	(wire (pts (xy 241.3000 162.5600) (xy 243.8400 162.5600))
 		(stroke (width 0) (type default)))
 	(wire (pts (xy 271.7800 146.0500) (xy 284.4800 146.0500))
@@
 	(junction (at 203.2000 36.8300) (diameter 0) (color 0 0 0 0))
 	(junction (at 228.6000 146.0500) (diameter 0) (color 0 0 0 0))
-	(junction (at 241.3000 146.0500) (diameter 0) (color 0 0 0 0))
-	(junction (at 241.3000 153.6700) (diameter 0) (color 0 0 0 0))
+	(junction (at 243.8400 162.5600) (diameter 0) (color 0 0 0 0))
 	(junction (at 284.4800 146.0500) (diameter 0) (color 0 0 0 0))
 	(junction (at 304.8000 36.8300) (diameter 0) (color 0 0 0 0))
@@
 			(effects (font (size 1.27 1.27)) (hide yes))))
 	(global_label "ST_PWR_EN" (shape passive)
-		(at 241.3000 156.2100 0)
-		(effects (font (size 1.27 1.27)) (justify left))
-		(property "Intersheetrefs" "${INTERSHEET_REFS}"
-			(at 241.3000 156.2100 0)
+		(at 241.3000 162.5600 180)
+		(effects (font (size 1.27 1.27)) (justify right))
+		(property "Intersheetrefs" "${INTERSHEET_REFS}"
+			(at 241.3000 162.5600 0)
 			(effects (font (size 1.27 1.27)) (hide yes))))
 	(label "CC1"
@@
 		(effects (font (size 2.0 2.0) (bold yes)) (justify left bottom))
 )
-	(text "Three things want the USB pair: the connector, the RP2350, the\neUSB2 repeater. The two switches join any two through the node\nUSB_X.\nUSB_SEL_CONN low, USB_SEL_MCU low: connector to RP2350 -- the\nboard as it powers up, both selects pulled down.\nCONN high: connector to repeater -- a host's USB goes over the\nair.\nMCU high: RP2350 to repeater -- the RP2350 is the device at the\nfar end.\nBoth high joins all three and is not a state to use.\nST_PWR_EN low turns the 1.8 V regulator off; it discharges its\noutput, which is a power-on reset for the ST60A3H1." (exclude_from_sim no)
+	(text "Three things want the USB pair: the connector, the RP2350, the\neUSB2 repeater. The two switches join any two through the node\nUSB_X.\nUSB_SEL_CONN low, USB_SEL_MCU low: connector to RP2350 -- the\nboard as it powers up, both selects pulled down.\nCONN high: connector to repeater -- a host's USB goes over the\nair.\nMCU high: RP2350 to repeater -- the RP2350 is the device at the\nfar end.\nBoth high joins all three and is not a state to use.\nST_PWR_EN high turns the 1.8 V regulator on; it is pulled down,\nso the rail is off until the RP2350 asks for it. Off, the\nregulator discharges its output, which is a power-on reset for\nthe ST60A3H1." (exclude_from_sim no)
 		(at 20.3200 194.3100 0)
 		(effects (font (size 1.27 1.27)) (justify left top))
